File: X14-Backplane.sch (EAGLE design)
At the start: 28 parts, among them J2 PXC-PTSM-04-RA-1778641, J3 PXC-8-RA-1778683, J8 PXC-8-RA-1778683

Commit message: second round of edits to bkplane
Connections:
- removed net ALERT1: U$10.14
- removed net ALERT2: U$10.12
- removed net SWCLK: U$10.8
- removed net SWDIO: U$10.6
- net ALERT_1: now also U$10.14
- net ALERT_2: now also U$10.12
- net NRST: no longer U$10.13
- net NRST_4: now also U$10.13
- net SWCLK_4: now also U$10.8
- net SWDIO_4: now also U$10.6
Changed lines of the file:
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@@
 <?xml version="1.0" encoding="utf-8"?>
 <!DOCTYPE eagle SYSTEM "eagle.dtd">
-<eagle version="9.6.2">
+<eagle version="9.5.0">
 <drawing>
 <settings>
@@
 <segment>
 <pinref part="U$5" gate="G$1" pin="12V"/>
-<wire x1="210.82" y1="144.78" x2="210.82" y2="152.4" width="0.1524" layer="91"/>
-<label x="210.82" y="152.4" size="1.778" layer="95"/>
+<wire x1="210.82" y1="144.78" x2="210.82" y2="153.67" width="0.1524" layer="91"/>
+<label x="209.55" y="153.67" size="1.778" layer="95"/>
 </segment>
 <segment>
 <pinref part="U$6" gate="G$1" pin="12V"/>
-<wire x1="223.52" y1="144.78" x2="223.52" y2="152.4" width="0.1524" layer="91"/>
-<label x="223.52" y="152.4" size="1.778" layer="95"/>
+<wire x1="223.52" y1="144.78" x2="223.52" y2="153.67" width="0.1524" layer="91"/>
+<label x="222.25" y="153.67" size="1.778" layer="95"/>
 </segment>
 <segment>
 <pinref part="U$7" gate="G$1" pin="12V"/>
-<wire x1="233.68" y1="144.78" x2="233.68" y2="152.4" width="0.1524" layer="91"/>
-<label x="233.68" y="152.4" size="1.778" layer="95"/>
+<wire x1="233.68" y1="144.78" x2="233.68" y2="153.67" width="0.1524" layer="91"/>
+<label x="232.41" y="153.67" size="1.778" layer="95"/>
 </segment>
 </net>
@@
 <junction x="243.84" y="60.96"/>
 </segment>
-<segment>
-<wire x1="33.02" y1="-99.06" x2="25.4" y2="-99.06" width="0.1524" layer="91"/>
-<label x="22.86" y="-99.06" size="1.778" layer="95"/>
-<pinref part="U$10" gate="G$1" pin="13"/>
-</segment>
 </net>
 <net name="ESCID_1" class="0">
@@
 <label x="99.5" y="39.4" size="1.778" layer="95"/>
 </segment>
+<segment>
+<wire x1="63.5" y1="-99.06" x2="73.66" y2="-99.06" width="0.1524" layer="91"/>
+<label x="68.58" y="-99.06" size="1.778" layer="95"/>
+<pinref part="U$10" gate="G$1" pin="14"/>
+</segment>
 </net>
 <net name="ALERT_2" class="0">
@@
 <label x="99.5" y="37" size="1.778" layer="95"/>
 </segment>
+<segment>
+<wire x1="73.66" y1="-96.52" x2="63.5" y2="-96.52" width="0.1524" layer="91"/>
+<label x="68.58" y="-96.52" size="1.778" layer="95"/>
+<pinref part="U$10" gate="G$1" pin="12"/>
+</segment>
 </net>
 <net name="CLK" class="0">
@@
 </net>
 <net name="12VGND" class="0">
-<segment>
-<pinref part="U$5" gate="G$1" pin="GND"/>
-<wire x1="210.82" y1="119.38" x2="210.82" y2="111.76" width="0.1524" layer="91"/>
-<label x="208.28" y="109.22" size="1.778" layer="95"/>
-</segment>
-<segment>
-<pinref part="U$6" gate="G$1" pin="GND"/>
-<wire x1="223.52" y1="119.38" x2="223.52" y2="111.76" width="0.1524" layer="91"/>
-<label x="220.98" y="109.22" size="1.778" layer="95"/>
-</segment>
-<segment>
-<pinref part="U$7" gate="G$1" pin="GND"/>
-<wire x1="233.68" y1="119.38" x2="233.68" y2="111.76" width="0.1524" layer="91"/>
-<label x="231.14" y="109.22" size="1.778" layer="95"/>
-</segment>
 <segment>
 <pinref part="DIST_TO_BACKPLANE" gate="G$1" pin="5"/>
@@
 <label x="15.24" y="43.18" size="1.778" layer="95" rot="R180"/>
 </segment>
+<segment>
+<pinref part="U$5" gate="G$1" pin="GND"/>
+<wire x1="210.82" y1="119.38" x2="210.82" y2="109.22" width="0.1524" layer="91"/>
+<label x="207.01" y="107.95" size="1.778" layer="95"/>
+</segment>
+<segment>
+<pinref part="U$6" gate="G$1" pin="GND"/>
+<wire x1="223.52" y1="119.38" x2="223.52" y2="109.22" width="0.1524" layer="91"/>
+<label x="220.98" y="107.95" size="1.778" layer="95"/>
+</segment>
+<segment>
+<pinref part="U$7" gate="G$1" pin="GND"/>
+<wire x1="233.68" y1="119.38" x2="233.68" y2="109.22" width="0.1524" layer="91"/>
+<label x="233.68" y="109.22" size="1.778" layer="95"/>
+</segment>
 </net>
 <net name="N$3" class="0">
@@
 <label x="203.2" y="45.72" size="1.778" layer="95"/>
 </segment>
+<segment>
+<pinref part="U$10" gate="G$1" pin="13"/>
+<wire x1="33.02" y1="-99.06" x2="24.13" y2="-99.06" width="0.1524" layer="91"/>
+<label x="22.86" y="-99.06" size="1.778" layer="95"/>
+</segment>
 </net>
 <net name="SWDIO_4" class="0">
@@
 <label x="12.7" y="90.17" size="1.778" layer="95"/>
 </segment>
+<segment>
+<wire x1="63.5" y1="-88.9" x2="73.66" y2="-88.9" width="0.1524" layer="91"/>
+<label x="68.58" y="-88.9" size="1.778" layer="95"/>
+<pinref part="U$10" gate="G$1" pin="6"/>
+</segment>
 </net>
 <net name="SWCLK_4" class="0">
@@
 <wire x1="50.8" y1="85.09" x2="60.96" y2="85.09" width="0.1524" layer="91"/>
 <label x="50.8" y="85.09" size="1.778" layer="95"/>
+</segment>
+<segment>
+<wire x1="63.5" y1="-91.44" x2="73.66" y2="-91.44" width="0.1524" layer="91"/>
+<label x="68.58" y="-91.44" size="1.778" layer="95"/>
+<pinref part="U$10" gate="G$1" pin="8"/>
 </segment>
 </net>
@@
 </segment>
 </net>
-<net name="SWDIO" class="0">
-<segment>
-<wire x1="63.5" y1="-88.9" x2="73.66" y2="-88.9" width="0.1524" layer="91"/>
-<label x="68.58" y="-88.9" size="1.778" layer="95"/>
-<pinref part="U$10" gate="G$1" pin="6"/>
-</segment>
-</net>
-<net name="SWCLK" class="0">
-<segment>
-<wire x1="63.5" y1="-91.44" x2="73.66" y2="-91.44" width="0.1524" layer="91"/>
-<label x="68.58" y="-91.44" size="1.778" layer="95"/>
-<pinref part="U$10" gate="G$1" pin="8"/>
-</segment>
-</net>
-<net name="ALERT2" class="0">
-<segment>
-<wire x1="73.66" y1="-96.52" x2="63.5" y2="-96.52" width="0.1524" layer="91"/>
-<label x="68.58" y="-96.52" size="1.778" layer="95"/>
-<pinref part="U$10" gate="G$1" pin="12"/>
-</segment>
-</net>
-<net name="ALERT1" class="0">
-<segment>
-<wire x1="63.5" y1="-99.06" x2="73.66" y2="-99.06" width="0.1524" layer="91"/>
-<label x="68.58" y="-99.06" size="1.778" layer="95"/>
-<pinref part="U$10" gate="G$1" pin="14"/>
-</segment>
-</net>
